Commit message: Real setup

File: drims_description/urdf/ur5e/ur5e_cell.urdf.xacro (robot description, xacro)
@@ -155,5 +155,12 @@
       >
       <origin xyz="${robot_xyz}" rpy="${robot_rpy}"/>
-  </xacro:ur_robot>
+    </xacro:ur_robot>
+    <link name="table_top_in_robot_origin"/>
+    <joint name="table_top_to_table_top_in_robot_origin" type="fixed">
+      <parent link="table_top"/>
+      <child link="table_top_in_robot_origin"/>
+      <!-- Same origin as the robot, but keep the table_top orientation. -->
+      <origin xyz="${robot_xyz}" rpy="0 0 0"/>
+    </joint>
   <!-- ========================================================= -->
   <!-- CAMERA FRAME -->
@@ -354,14 +361,14 @@
     </joint>
   </xacro:macro>
-  <xacro:safety_barrier name="barrier_back" parent="base_link"
+  <xacro:safety_barrier name="barrier_back" parent="table_top_in_robot_origin"
     xyz="${barrier_back_offset}"
     size="0.1 ${table_width} 0.8"/>
-  <xacro:safety_barrier name="barrier_left" parent="base_link"
+  <xacro:safety_barrier name="barrier_left" parent="table_top_in_robot_origin"
     xyz="${barrier_left_offset}"
     size="${table_length} 0.1 0.8"/>
-  <xacro:safety_barrier name="barrier_right" parent="base_link"
+  <xacro:safety_barrier name="barrier_right" parent="table_top_in_robot_origin"
     xyz="${barrier_right_offset}"
     size="${table_length} 0.1 0.8"/>
-  <xacro:safety_barrier name="barrier_top" parent="base_link"
+  <xacro:safety_barrier name="barrier_top" parent="table_top_in_robot_origin"
     xyz="${barrier_top_offset}"
     size="${table_length} ${table_width} 0.1"/>

Commit message: Fix real hardware for first, and third cell

File: drims_description/urdf/ur5e/ur5e_cell.urdf.xacro (robot description, xacro)
@@ -278,5 +278,5 @@
         </geometry>
         <material name="gray_transparent"/>
-        <origin xyz="${beam/2} ${beam/2+frame_y/2} ${post_height/2}" rpy="0 0 0"/>
+        <origin xyz="${beam/2} ${frame_y/2} ${post_height/2}" rpy="0 0 0"/>
       </visual>
       <collision>
@@ -285,5 +285,5 @@
         </geometry>
         <material name="red_transparent"/>
-        <origin xyz="${beam/2} ${beam/2+frame_y/2} ${post_height/2}" rpy="0 0 0"/>
+        <origin xyz="${beam/2} ${frame_y/2} ${post_height/2}" rpy="0 0 0"/>
       </collision>
     </link>
@@ -294,4 +294,28 @@
     </joint>
     <!-- ======================================================= -->
+    <!-- FLOOR -->
+    <!-- ======================================================= -->
+    <link name="${name}_floor">
+      <visual>
+        <geometry>
+          <box size="${frame_x - 2*beam} ${frame_y - 2*beam} 0.005"/>
+        </geometry>
+        <material name="gray_transparent"/>
+        <origin xyz="${frame_x/2} ${frame_y/2} 0.0025" rpy="0 0 0"/>
+      </visual>
+      <collision>
+        <geometry>
+          <box size="${frame_x - 2*beam} ${frame_y - 2*beam} 0.005"/>
+        </geometry>
+        <material name="gray_transparent"/>
+        <origin xyz="${frame_x/2} ${frame_y/2} 0.0025" rpy="0 0 0"/>
+      </collision>
+    </link>
+    <joint name="${name}_floor_joint" type="fixed">
+      <parent link="${name}_post"/>
+      <child link="${name}_floor"/>
+      <origin xyz="0 0 0" rpy="0 0 0"/>
+    </joint>
+    <!-- ======================================================= -->
     <!-- TOP HORIZONTAL CAMERA BAR -->
     <!-- ======================================================= -->
@@ -302,12 +326,12 @@
         </geometry>
         <material name="gray_transparent"/>
-        <origin xyz="${frame_x/2} ${beam/2+frame_y/2} ${post_height}" rpy="0 0 0"/>
-      </visual>
-      <collision>
-        <geometry>
-          <box size="${frame_x} ${beam} ${beam}"/>
-        </geometry>
-        <material name="red_transparent"/>
-        <origin xyz="${frame_x/2} ${beam/2+frame_y/2} ${post_height}" rpy="0 0 0"/>
+        <origin xyz="${frame_x/2} ${frame_y/2} ${post_height}" rpy="0 0 0"/>
+      </visual>
+      <collision>
+        <geometry>
+          <box size="${frame_x} ${beam} ${beam}"/>
+        </geometry>
+        <material name="red_transparent"/>
+        <origin xyz="${frame_x/2} ${frame_y/2} ${post_height}" rpy="0 0 0"/>
       </collision>
     </link>
@@ -315,4 +339,28 @@
       <parent link="${name}_post"/>
       <child link="${name}_top_bar"/>
+      <origin xyz="0 0 0" rpy="0 0 0"/>
+    </joint>
+    <!-- ======================================================= -->
+    <!-- TOP-LATERAL HORIZONTAL CAMERA BAR -->
+    <!-- ======================================================= -->
+    <link name="${name}_top_bar_camera">
+      <visual>
+        <geometry>
+          <box size="${frame_x/2} ${beam*2} ${beam+0.025}"/>
+        </geometry>
+        <material name="gray_transparent"/>
+        <origin xyz="${frame_x/2} ${frame_y/2} ${post_height-0.025}" rpy="0 0 0"/>
+      </visual>
+      <collision>
+        <geometry>
+          <box size="${frame_x/2} ${beam*2} ${beam+0.025}"/>
+        </geometry>
+        <material name="red_transparent"/>
+        <origin xyz="${frame_x/2} ${frame_y/2} ${post_height-0.025}" rpy="0 0 0"/>
+      </collision>
+    </link>
+    <joint name="${name}_top_bar_camera_joint" type="fixed">
+      <parent link="${name}_post"/>
+      <child link="${name}_top_bar_camera"/>
       <origin xyz="0 0 0" rpy="0 0 0"/>
     </joint>
@@ -323,9 +371,9 @@
     xyz="${camera_frame_xyz}"
     rpy="${camera_frame_rpy}"
-    frame_x="0.8"
-    frame_y="0.6"
+    frame_x="0.73"
+    frame_y="0.53"
     beam="0.05"
     height="0.7"
-    post_height="0.8"/>
+    post_height="0.67"/>
   <!-- ========================================================= -->
   <!-- CAMERA -->

Commit message: fix tip for drims fingers

File: drims_description/urdf/ur5e/ur5e_cell.urdf.xacro (robot description, xacro)
@@ -395,5 +395,5 @@
     <parent link="tool0"/>
     <child link="tip"/>
-    <origin xyz="0 0 0.15" rpy="0 0 0"/>
+    <origin xyz="0 0 0.17" rpy="0 0 0"/>
   </joint>
 </robot>
